Commit message: initial release ready to go

File: env/bullet_world/urdfs/human.urdf (robot description, URDF)
Before this commit: robot urdf_robot, 1 links, 0 joints
Links:
- link base_link: geometry collision sphere radius=0.1; visual mesh filename=textured_sphere_smooth.obj scale=0.1 0.1 0.1

File: env/bullet_world/urdfs/robot_goal.urdf (robot description, URDF)
Before this commit: robot urdf_robot, 1 links, 0 joints
Links:
- link base_link: geometry visual mesh filename=textured_sphere_smooth.obj scale=0.2 0.2 0.2
