Commit message: modify franka dh parameter to include hand

File: env/bullet_world/urdfs/human_goal.urdf (robot description, URDF)
Before this commit: robot urdf_robot, 1 links, 0 joints
Links:
- link base_link: geometry visual mesh filename=textured_sphere_smooth.obj scale=0.05 0.05 0.05

File: env/bullet_world/urdfs/robot_goal.urdf (robot description, URDF)
Before this commit: robot urdf_robot, 1 links, 0 joints
Links:
- link base_link: geometry visual mesh filename=textured_sphere_smooth.obj scale=0.05 0.05 0.05
